File: display.kicad_sch (KiCad schematic)
At the start: 7 parts, among them J16 Oled SSD1306 128x32, J17 Adafruit ST7789, U5 ER_OLEDM0.91_1x-I2C

Commit message: se agrego osciloscoio
Other:
- moved on the sheet: R39, R40
Changed lines of the file:
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@@
 	(wire
 		(pts
-			(xy 110.49 134.62) (xy 110.49 138.43)
+			(xy 104.14 142.24) (xy 104.14 146.05)
 		)
 		(stroke
@@
 	(wire
 		(pts
-			(xy 96.52 138.43) (xy 110.49 138.43)
+			(xy 90.17 146.05) (xy 104.14 146.05)
 		)
 		(stroke
@@
 	(wire
 		(pts
-			(xy 83.82 124.46) (xy 96.52 124.46)
+			(xy 77.47 132.08) (xy 90.17 132.08)
 		)
 		(stroke
@@
 	)
 	(label "SDA"
-		(at 104.14 138.43 180)
+		(at 97.79 146.05 180)
 		(effects
 			(font
@@
 	)
 	(label "SCL"
-		(at 88.9 124.46 180)
+		(at 82.55 132.08 180)
 		(effects
 			(font
@@
 	(hierarchical_label "SDA"
 		(shape input)
-		(at 96.52 138.43 180)
+		(at 90.17 146.05 180)
 		(effects
 			(font
@@
 	(hierarchical_label "SCL"
 		(shape input)
-		(at 83.82 124.46 180)
+		(at 77.47 132.08 180)
 		(effects
 			(font
@@
 	(symbol
 		(lib_id "Device:R")
-		(at 110.49 130.81 0)
+		(at 104.14 138.43 0)
 		(unit 1)
 		(body_style 1)
@@
 		(fields_autoplaced yes)
 		(property "Reference" "R40"
-			(at 113.03 129.5399 0)
+			(at 106.68 137.1599 0)
 			(show_name no)
 			(do_not_autoplace no)
@@
 		)
 		(property "Value" "2k2"
-			(at 113.03 132.0799 0)
+			(at 106.68 139.6999 0)
 			(show_name no)
 			(do_not_autoplace no)
@@
 		)
 		(property "Footprint" "Resistor_SMD:R_0805_2012Metric"
-			(at 108.712 130.81 90)
+			(at 102.362 138.43 90)
 			(hide yes)
 			(show_name no)
@@
 		)
 		(property "Datasheet" ""
-			(at 110.49 130.81 0)
+			(at 104.14 138.43 0)
 			(hide yes)
 			(show_name no)
@@
 		)
 		(property "Description" ""
-			(at 110.49 130.81 0)
+			(at 104.14 138.43 0)
 			(show_name no)
 			(do_not_autoplace no)
@@
 	(symbol
 		(lib_id "Device:R")
-		(at 96.52 120.65 0)
+		(at 90.17 128.27 0)
 		(unit 1)
 		(body_style 1)
@@
 		(fields_autoplaced yes)
 		(property "Reference" "R39"
-			(at 99.06 119.3799 0)
+			(at 92.71 126.9999 0)
 			(show_name no)
 			(do_not_autoplace no)
@@
 		)
 		(property "Value" "2k2"
-			(at 99.06 121.9199 0)
+			(at 92.71 129.5399 0)
 			(show_name no)
 			(do_not_autoplace no)
@@
 		)
 		(property "Footprint" "Resistor_SMD:R_0805_2012Metric"
-			(at 94.742 120.65 90)
+			(at 88.392 128.27 90)
 			(hide yes)
 			(show_name no)
@@
 		)
 		(property "Datasheet" ""
-			(at 96.52 120.65 0)
+			(at 90.17 128.27 0)
 			(hide yes)
 			(show_name no)
@@
 		)
 		(property "Description" ""
-			(at 96.52 120.65 0)
+			(at 90.17 128.27 0)
 			(show_name no)
 			(do_not_autoplace no)
@@
 	(symbol
 		(lib_id "power:+3V3")
-		(at 96.52 116.84 0)
+		(at 90.17 124.46 0)
 		(unit 1)
 		(body_style 1)
@@
 		(fields_autoplaced yes)
 		(property "Reference" "#PWR068"
-			(at 96.52 120.65 0)
+			(at 90.17 128.27 0)
 			(hide yes)
 			(show_name no)
@@
 		)
 		(property "Value" "+3V3"
-			(at 96.52 111.76 0)
+			(at 90.17 119.38 0)
 			(show_name no)
 			(do_not_autoplace no)
@@
 		)
 		(property "Footprint" ""
-			(at 96.52 116.84 0)
+			(at 90.17 124.46 0)
 			(hide yes)
 			(show_name no)
@@
 		)
 		(property "Datasheet" ""
-			(at 96.52 116.84 0)
+			(at 90.17 124.46 0)
 			(hide yes)
 			(show_name no)
@@
 		)
 		(property "Description" "Power symbol creates a global label with name \"+3V3\""
-			(at 96.52 116.84 0)
+			(at 90.17 124.46 0)
 			(hide yes)
 			(show_name no)
@@
 	(symbol
 		(lib_id "power:+3V3")
-		(at 110.49 127 0)
+		(at 104.14 134.62 0)
 		(unit 1)
 		(body_style 1)
@@
 		(fields_autoplaced yes)
 		(property "Reference" "#PWR069"
-			(at 110.49 130.81 0)
+			(at 104.14 138.43 0)
 			(hide yes)
 			(show_name no)
@@
 		)
 		(property "Value" "+3V3"
-			(at 110.49 121.92 0)
+			(at 104.14 129.54 0)
 			(show_name no)
 			(do_not_autoplace no)
@@
 		)
 		(property "Footprint" ""
-			(at 110.49 127 0)
+			(at 104.14 134.62 0)
 			(hide yes)
 			(show_name no)
@@
 		)
 		(property "Datasheet" ""
-			(at 110.49 127 0)
+			(at 104.14 134.62 0)
 			(hide yes)
 			(show_name no)
@@
 		)
 		(property "Description" "Power symbol creates a global label with name \"+3V3\""
-			(at 110.49 127 0)
-			(hide yes)
-			(show_name no)
+			(at 104.14 134.62 0)
+			(hide yes)
+			(show_name no)
