File: ft232.kicad_sch (KiCad schematic)
At the start: 58 parts, among them J1 tp, J10 tp, J11 FT232RL, J12 tp_ft232_, J13 USB_B_Mini, J14 tp_ft232_, J2 tp, J3 tp, J4 tp, J5 tp, J6 tp, J7 tp, J8 tp, J9 tp, Q1 FDN306P, Q2 2N7002, Q3 2N7002, U1 FT232BM, U2 93CxxA, U3 LM1117DT-3.3, Y1 Crystal

Commit message: se agrego osciloscoio
Parts:
- removed C1, C12, C13, C2, C3, C4, C5, C6, C7: 100nf, Capacitor_SMD:C_0805_2012Metric, symbol Device:C
- removed C10, C8: 15p, Capacitor_SMD:C_0805_2012Metric, symbol Device:C
- removed C11, C9: 33nf, Capacitor_SMD:C_0805_2012Metric, symbol Device:C
- removed D1, D2: RX, Diode_SMD:D_0805_2012Metric, symbol Device:LED_Small
- removed J1, J2, J3, J4, J5, J6, J7, J8, J9: tp, TestPoint:TestPoint_Pad_D1.5mm, symbol Connector:Conn_01x01_Pin
- removed J10: tp, TestPoint:TestPoint_THTPad_2.0x2.0mm_Drill1.0mm, symbol Connector:Conn_01x01_Pin
- removed J11: FT232RL, Connector_PinHeader_2.54mm:PinHeader_1x06_P2.54mm_Vertical, symbol Connector:Conn_01x06_Pin
- removed J12, J14: tp_ft232_, Library:connector_pin1, symbol Connector:Conn_01x01_Pin
- removed J13: USB_B_Mini, kiC:USB_Mini-B_Lumberg_2486_01_Horizontal, symbol Connector:USB_B_Mini
- removed JP6, JP7: Jumper_Open, Jumper:SolderJumper-2_P1.3mm_Open_RoundedPad1.0x1.5mm, symbol Jumper:Jumper_2_Open
- removed L1: 100mh, Inductor_SMD:L_1206_3216Metric, symbol Device:L
- removed Q1: FDN306P, Package_TO_SOT_SMD:SOT-23W, symbol FDN306P:FDN306P
- removed Q2, Q3: 2N7002, Package_TO_SOT_SMD:SOT-23, symbol Transistor_FET:2N7002
- removed R1, R17, R2, R3, R4: 2k2, Resistor_SMD:R_0805_2012Metric, symbol Device:R
- removed R10, R11, R14, R15, R5, R7: 10K, Resistor_SMD:R_0805_2012Metric, symbol Device:R
- removed R12, R13: 1K5, Resistor_SMD:R_0805_2012Metric, symbol Device:R
- removed R16: 4K7, Resistor_SMD:R_0805_2012Metric, symbol Device:R
- removed R18, R19: 27, Resistor_SMD:R_0805_2012Metric, symbol Device:R
- removed R6: 10K, Resistor_SMD:R_0603_1608Metric, symbol Device:R
- removed R8, R9: 100, Resistor_SMD:R_0805_2012Metric, symbol Device:R
- removed U1: FT232BM, Package_QFP:LQFP-32_7x7mm_P0.8mm, symbol Interface_USB:FT232BM
- removed U2: 93CxxA, Package_SO:SOIC-8_5.3x5.3mm_P1.27mm, symbol Memory_EEPROM:93CxxA
- removed U3: LM1117DT-3.3, kiC:SOT-223-3_TabPin2, symbol Regulator_Linear:LM1117DT-3.3
- removed Y1: Crystal, Crystal:Resonator-2Pin_W10.0mm_H5.0mm, symbol Device:Crystal
Other:
- note removed: "DTR RTS -> EN IO9 1 1 1 1 0 0 1 1 1 0 0 1 0 1 1 0"
