File: max98357a.kicad_sch (KiCad schematic)
At the start: 16 parts, among them U4 MAX98357A

Commit message: se agrego osciloscoio
Parts:
- removed JP10: 0, Jumper:SolderJumper-2_P1.3mm_Open_RoundedPad1.0x1.5mm, symbol Jumper:Jumper_2_Open
Connections:
- net GNDA is gone; now on net GND: C15.1, C16.1, C17.1, C18.1, J15.6 (Pin_6), R23.2, U4.11 (GND), U4.15 (GND), U4.17 (PAD), U4.3 (GND)
