File: pico_hw_dev.kicad_pcb (KiCad board)
At the start: 2 copper layers, 99.1 x 111.9 mm, 220 parts, among them J1 tp, J10 tp, J11 FT232RL, J13 USB_B_Mini, J16 Oled SSD1306 128x32, J17 Adafruit ST7789, J18 Micro_SD_Card, J19 USB_B_Mini, J2 tp, J20 gpio_rp2040, J21 gpio_rp2040, J22 gpio_rp2040, J23 gpio_rp2040, J24 gpio_rp2040, J25 gpio_rp2040, J3 tp, J4 tp, J48 logic_convert, J49 DE15_Pins_HighDensity, J5 tp, J50 Mini-DIN-6, J6 tp, J7 tp, J8 tp, J9 tp, Q1 FDN306P, Q10 2N7002, Q2 2N7002, Q3 2N7002, Q4 2N7002, Q5 Q_NPN_BCE, Q6 FDN306P, Q7 Q_NPN_BCE, Q8 FDN306P, Q9 2N7002, SW1 up, SW2 down, SW3 left, SW4 rigth, SW5 up, SW6 down, SW7 run, SW8 run, U1 FT232BM, U2 93CxxA, U3 LM1117DT-3.3, U4 MAX98357A, U5 ER_OLEDM0.91_1x-I2C, U6 RP2040, U7 R-78E3.3-0.5, U8 TXS0108EPW, U9 W25Q16JVSS, Y1 Crystal, Y2 Crystal_GND24_Small

Commit message: Update KiCad project files
Parts:
- added J27: picoprobe debugger, Connector_PinHeader_2.54mm:PinHeader_1x07_P2.54mm_Vertical, F.Cu at (58.7, 102.8)
- A1: footprint Module:RaspberryPi_Pico_Common_THT -> kiC:RaspberryPi_Pico
- moved R50 69.8 mm to (98.2, 97.8)
- moved C42 59.9 mm to (86.3, 66.4), turned to 90 degrees
- moved C40 52.8 mm to (78.4, 83.0)
- moved C37 52.5 mm to (78.9, 71.6), turned to 90 degrees
- moved C43 49.3 mm to (75.5, 87.4)
- moved C47 47.5 mm to (78.6, 68.2), turned to 90 degrees
- moved C48 47.5 mm to (78.4, 77.3)
- moved R47 41.9 mm to (71.1, 65.6), turned to -90 degrees
- moved C41 40.0 mm to (67.0, 69.5), turned to -90 degrees
- moved C45 38.2 mm to (67.3, 77.6)
- moved R48 37.8 mm to (72.9, 65.6), turned to -90 degrees
- moved C44 37.3 mm to (67.0, 72.9), turned to 90 degrees
- moved C49 37.0 mm to (67.5, 81.8)
- moved C46 36.0 mm to (67.1, 66.2), turned to 90 degrees
- moved A1 26.6 mm to (72.7, 79.3)
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Connections:
- net /picohw/GPIO_10 renamed /IO_10
- net /picohw/GPIO_12 renamed /IO_12
- net /picohw/GPIO_13 renamed /IO_13
- net /picohw/GPIO_14 renamed /IO_14
- net /picohw/GPIO_15 renamed /IO_15
- net /picohw/GPIO_22 renamed /IO_22
- net /picohw/GPIO_23 renamed /IO_23
- net /picohw/GPIO_24 renamed /IO_24
- net /picohw/GPIO_25 renamed /IO_25
- net /picohw/GPIO_4 renamed /IO_4
- net /picohw/GPIO_5 renamed /IO_5
- net /picohw/GPIO_6 renamed /IO_6
- net /picohw/GPIO_7 renamed /IO_7
- net /picohw/adc_0_rp2040 renamed /ADC_0
- net /picohw/adc_1_rp2040 renamed /ADC_1
- net /picohw/adc_2_rp2040 renamed /ADC_2
- A1 pad 13: Net-(A1-GND-Pad13) -> GND
- A1 pad 18: Net-(A1-GND-Pad13) -> GND
- A1 pad 21: /picohw/GPIO_16 -> /MISO
- A1 pad 23: Net-(A1-GND-Pad13) -> GND
- A1 pad 27: /picohw/GPIO_21 -> /SCL_I2C
- A1 pad 28: Net-(A1-GND-Pad13) -> GND
- A1 pad 3: Net-(A1-GND-Pad13) -> GND
- A1 pad 33: unconnected-(A1-AGND-Pad33) -> GND
- A1 pad 38: Net-(A1-GND-Pad13) -> GND
- A1 pad 8: Net-(A1-GND-Pad13) -> GND
- D4 pad 2: /CS -> CS_RP2040
- J16 pad 3: /SDA_I2C -> MISO_RP_2040
- J18 pad 1: /MSCK -> MSCLK_RP_2040
- J18 pad 2: /CS -> CS_RP2040
- J18 pad 7: /MOSI -> MOSI_RP_2040
- R40 pad 2: /SDA_I2C -> MISO_RP_2040
- R43 pad 2: /CS -> CS_RP2040
- R44 pad 1: /MOSI -> MOSI_RP_2040
- R45 pad 2: /MSCK -> MSCLK_RP_2040
- U5 pad 4: /SDA_I2C -> MISO_RP_2040
- U6 pad 27: /picohw/GPIO_16 -> /MISO
- U6 pad 32: /picohw/GPIO_21 -> /SCL_I2C

Commit message: se agrego osciloscoio
Parts:
- removed C10, C8: 15p, Capacitor_SMD:C_0805_2012Metric
- removed C11, C9: 33nf, Capacitor_SMD:C_0805_2012Metric
- removed C12, C13, C3, C6, C7: 100nf, Capacitor_SMD:C_0805_2012Metric
- removed D1, D2: RX, Diode_SMD:D_0805_2012Metric
- removed J10: tp, TestPoint:TestPoint_THTPad_2.0x2.0mm_Drill1.0mm
- removed J11: FT232RL, Connector_PinHeader_2.54mm:PinHeader_1x06_P2.54mm_Vertical
- removed J13: USB_B_Mini, kiC:USB_Mini-B_Lumberg_2486_01_Horizontal
- removed J48: logic_convert, Connector_PinHeader_2.54mm:PinHeader_2x05_P2.54mm_Vertical
- removed J49: DE15_Pins_HighDensity, Library:AMPHENOL_L77HDE15SD1CH4RHNVGA
- removed J5, J6, J7, J8, J9: tp, TestPoint:TestPoint_Pad_D1.5mm
- removed JP1, JP2, JP3, JP4, JP5, JP6, JP7: Jumper_Open, Jumper:SolderJumper-2_P1.3mm_Open_RoundedPad1.0x1.5mm
- removed JP10: 0, Jumper:SolderJumper-2_P1.3mm_Open_RoundedPad1.0x1.5mm
- removed L1: 100mh, Inductor_SMD:L_1206_3216Metric
- removed MK1: INMP441ACEZ-R7, kiC:MIC_INMP441ACEZ-R7
- removed Q1: FDN306P, Package_TO_SOT_SMD:SOT-23W
- removed Q2, Q3: 2N7002, Package_TO_SOT_SMD:SOT-23
- removed R1, R17, R2, R3, R4: 2k2, Resistor_SMD:R_0805_2012Metric
- removed R10, R11, R14, R15, R5, R7: 10K, Resistor_SMD:R_0805_2012Metric
- removed R12, R13: 1K5, Resistor_SMD:R_0805_2012Metric
- removed R16: 4K7, Resistor_SMD:R_0805_2012Metric
- removed R18, R19: 27, Resistor_SMD:R_0805_2012Metric
- removed R6: 10K, Resistor_SMD:R_0603_1608Metric
- removed R63, R69, R75: 2K, Resistor_SMD:R_0805_2012Metric
- removed R64, R70, R76: 1K, Resistor_SMD:R_0805_2012Metric
- removed R65, R71, R77: 500, Resistor_SMD:R_0805_2012Metric
- removed R66, R72: 16K, Resistor_SMD:R_0805_2012Metric
- removed R67, R73: 8K, Resistor_SMD:R_0805_2012Metric
- removed R68, R74: 4K, Resistor_SMD:R_0805_2012Metric
- removed R78, R79: 120, Resistor_SMD:R_0805_2012Metric
- removed R8, R9: 100, Resistor_SMD:R_0805_2012Metric
- removed U1: FT232BM, Package_QFP:LQFP-32_7x7mm_P0.8mm
- removed U2: 93CxxA, Package_SO:SOIC-8_5.3x5.3mm_P1.27mm
- removed U3: LM1117DT-3.3, kiC:SOT-223-3_TabPin2
- removed Y1: Crystal, Crystal:Resonator-2Pin_W10.0mm_H5.0mm
- added J26: FT232RL, Connector_PinHeader_2.54mm:PinHeader_1x06_P2.54mm_Vertical, F.Cu at (58.6, 64.9)
- added JP13: NL, Jumper:SolderJumper-2_P1.3mm_Open_RoundedPad1.0x1.5mm, B.Cu at (90.5, 104.7)
- added JP14: NL, Jumper:SolderJumper-2_P1.3mm_Open_RoundedPad1.0x1.5mm, B.Cu at (94.0, 104.7)
- added U10: W25Q16JVSS, kiC:Winbond_XSON-8-1EP_4x4mm_P0.8mm_EP2.3x3.0mm, F.Cu at (73.5, 92.8)
- C2: moved to F.Cu
- J1, J3, J4: value tp -> Conn_Coaxial; footprint TestPoint:TestPoint_Pad_D1.5mm -> Connector_Coaxial:SMA_BAT_Wireless_BWSMA-KWE-Z001; moved to F.Cu
- J2: value tp -> LOGIC; footprint TestPoint:TestPoint_Pad_D1.5mm -> Connector_PinHeader_2.54mm:PinHeader_1x10_P2.54mm_Vertical; moved to F.Cu
- R60: value 16K -> 10k
- R61: value 8K -> 10k
- R62: value 4K -> 10k
- SW7: value run -> boot; footprint Button_Switch_SMD:SW_SPST_B3U-1000P -> Button_Switch_SMD:SW_SPST_CK_RS282G05A3
- moved J1 69.3 mm to (150.5, 73.8), turned to -90 degrees
- moved J3 65.8 mm to (150.5, 85.4), turned to -90 degrees
- moved U8 64.4 mm to (109.3, 140.5)
- moved J4 55.6 mm to (150.5, 97.0), turned to -90 degrees
- moved D7 38.3 mm to (115.2, 132.9)
- moved D3 38.3 mm to (112.3, 132.9)
- moved D4 38.3 mm to (109.3, 132.9)
- moved D5 38.3 mm to (106.4, 132.9)
- moved D6 38.3 mm to (103.4, 132.9)
- moved R26 38.3 mm to (112.2, 128.4)
- moved R27 38.3 mm to (109.3, 128.4)
- moved R28 38.3 mm to (106.3, 128.4)
- moved R29 38.3 mm to (103.4, 128.4)
- moved R30 38.3 mm to (115.2, 128.5)
- moved C1 23.9 mm to (93.0, 128.5), turned to 0 degrees
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Connections:
- net /picohw/swclk renamed /swclk
- net /picohw/swdio renamed /swdio
- net /vga/GP_0 renamed /osciloscope/CH1
- net /vga/GP_1 renamed /osciloscope/CH2
- net /vga/GP_2 renamed /osciloscope/CH3
- A1 pad 16: /IO_12 -> SD
- A1 pad 19: /IO_14 -> CLK_ST7789
- A1 pad 20: /IO_15 -> DI_ST7789
- A1 pad 26: MISO_RP_2040 -> RES_ST7789
- A1 pad 27: /SCL_I2C -> DC_ST7789
- A1 pad 29: /IO_22 -> BLK_ST7789
- C1 pad 1: +3.3VA -> +3.3V
- C1 pad 2: GND1 -> GND
- C15 pad 1: GNDA -> GND
- C16 pad 1: GNDA -> GND
- C17 pad 1: GNDA -> GND
- C18 pad 1: GNDA -> GND
- C2 pad 1: +3.3VA -> +3.3V
- C2 pad 2: GND1 -> GND
- C20 pad 1: /IO_19 -> /IO_7
- C21 pad 1: /IO_11 -> /IO_13
- C23 pad 1: RX_RP2040 -> /IO_24
- C24 pad 1: TX_RP2040 -> /IO_23
- C4 pad 1: GND1 -> GND
- C4 pad 2: +3.3VA -> +3.3V
- C5 pad 1: GND1 -> GND
- C5 pad 2: +3.3VA -> +3.3V
- D3 pad 2: /IO_8 -> TX_RP2040
- D4 pad 2: CS_RP2040 -> RX_RP2040
- D5 pad 2: /L/R -> /IO_5
- D6 pad 2: /OE -> /IO_6
- J1 pad 1: /ft232/FT_RST -> Net-(J1-In)
- J15 pad 1: /WS -> /IO_4
- J15 pad 2: /SCK -> SCL_RPI
- J15 pad 3: /DIN -> SDA_RPI
- J15 pad 6: GNDA -> GND
- J16 pad 3: MISO_RP_2040 -> RES_ST7789
- J16 pad 5: /SCL_I2C -> DC_ST7789
- J2 pad 1: /ft232/FT_CTS -> /Logic_convert/vcc
- J27 pad 6: RX_RP2040 -> /debugger/GPIO_1
- J27 pad 7: TX_RP2040 -> /debugger/GPIO_0
- J3 pad 1: /ft232/FT_DTR -> Net-(J3-In)
- J4 pad 1: /ft232/FT_DRS -> Net-(J4-In)
- J50 pad 1: /ps2/keyboard_data -> /ADC_0
- J50 pad 5: /ps2/clock -> /ADC_1
- JP8 pad 1: /L/R -> GND
- JP9 pad 2: /L/R -> GND
- MK2 pad 1: /SCK -> /IO_10
- MK2 pad 3: /WS -> /IO_11
- MK2 pad 4: /L/R -> GND
- MK3 pad 1: /SCK -> /IO_10
- MK3 pad 3: /WS -> /IO_11
- MK3 pad 4: /L/R -> GND
- Q10 pad 2: /ps2/keyboard_data -> /ADC_0
- Q10 pad 3: /ps2/keyboard_data -> /ADC_0
- Q4 pad 2: /IO_8 -> /WS2812
- Q6 pad 1: /OE -> /WS2812
- Q9 pad 1: /OE -> /WS2812
- R20 pad 1: /L/R -> GND
- R23 pad 2: GNDA -> GND
- R32 pad 2: /IO_19 -> /IO_7
- R33 pad 2: /IO_11 -> /IO_13
- R35 pad 2: RX_RP2040 -> /IO_24
- R36 pad 2: TX_RP2040 -> /IO_23
- R37 pad 1: /IO_8 -> /WS2812
- R39 pad 2: /SCL_I2C -> DC_ST7789
- R40 pad 2: MISO_RP_2040 -> RES_ST7789
- R52 pad 1: /OE -> /Logic_convert/OE
- R54 pad 2: /OE -> /WS2812
- R58 pad 1: /ps2/keyboard_data -> /ADC_0
- R59 pad 1: /ps2/keyboard_data -> /ADC_0
- R60 pad 1: /vga/RED -> Net-(J1-In)
- R61 pad 1: /vga/RED -> Net-(J3-In)
- R62 pad 1: /vga/RED -> Net-(J4-In)
- SW1 pad 1: /IO_19 -> /IO_7
- SW4 pad 1: /IO_11 -> /IO_13
- SW5 pad 1: TX_RP2040 -> /IO_23
- SW6 pad 1: RX_RP2040 -> /IO_24
- U4 pad 1: /DIN -> SDA_RPI
- U4 pad 11: GNDA -> GND
- U4 pad 14: /WS -> /IO_4
- U4 pad 15: GNDA -> GND
- U4 pad 16: /SCK -> SCL_RPI
- U4 pad 17: GNDA -> GND
- U4 pad 3: GNDA -> GND
- U5 pad 3: /SCL_I2C -> DC_ST7789
- U5 pad 4: MISO_RP_2040 -> RES_ST7789
- U6 pad 15: /IO_12 -> SD
- U6 pad 17: /IO_14 -> CLK_ST7789
- U6 pad 18: /IO_15 -> DI_ST7789
- U6 pad 31: MISO_RP_2040 -> RES_ST7789
- U6 pad 32: /SCL_I2C -> DC_ST7789
- U6 pad 34: /IO_22 -> BLK_ST7789
- U8 pad 1: /IO_19 -> TX_RP2040
- U8 pad 3: /IO_8 -> RX_RP2040
- U8 pad 4: /IO_9 -> /IO_5
- U8 pad 5: /IO_11 -> /IO_6
- U8 pad 6: RX_RP2040 -> /IO_7
- U8 pad 7: /IO_18 -> /IO_8
- U8 pad 8: TX_RP2040 -> /IO_9
- U8 pad 9: /Logic_convert/A8 -> /IO_13
