File: pico_hw_dev.kicad_sch (KiCad schematic)
At the start: 5 parts

Commit message: Update KiCad project files
Other:
- sheet picohw ports: added SWCLK, SWDIO; removed none

Commit message: se agrego osciloscoio
Parts:
- removed JP1, JP2, JP3, JP4, JP5: Jumper_Open, Jumper:SolderJumper-2_P1.3mm_Open_RoundedPad1.0x1.5mm, symbol Jumper:Jumper_2_Open
- added JP13, JP14: NL, Jumper:SolderJumper-2_P1.3mm_Open_RoundedPad1.0x1.5mm, symbol Jumper:Jumper_2_Open
Connections:
- net ADC_3: now also JP14.1 (A)
- net IO_25: now also JP13.1 (A)
- new net WS2812: JP13.2 (B), JP14.2 (B)
Other:
- removed sheet ft232
- removed sheet vga
- added sheet debugger (debugger.kicad_sch)
- added sheet osciloscope (osciloscope.kicad_sch)
- sheet Logic_convert ports: added CONTROL; removed none
