File: picohw.kicad_sch (KiCad schematic)
At the start: 35 parts, among them J19 USB_B_Mini, J20 gpio_rp2040, J21 gpio_rp2040, J22 gpio_rp2040, J23 gpio_rp2040, J24 gpio_rp2040, J25 gpio_rp2040, SW7 run, SW8 run, U6 RP2040, U7 R-78E3.3-0.5, U9 W25Q16JVSS, Y2 Crystal_GND24_Small

Commit message: Update KiCad project files
Parts:
- added J27: picoprobe debugger, Connector_PinHeader_2.54mm:PinHeader_1x07_P2.54mm_Vertical, symbol Connector:Conn_01x07_Pin
- A1: footprint Module:RaspberryPi_Pico_Common_THT -> kiC:RaspberryPi_Pico
Connections:
- net GND: now also A1.13 (GND), A1.18 (GND), A1.23 (GND), A1.28 (GND), A1.3 (GND), A1.33 (AGND), A1.38 (GND), A1.8 (GND), J27.3 (Pin_3)
- net RX_RP2040: now also J27.6 (Pin_6)
- net TX_RP2040: now also J27.7 (Pin_7)
- net swclk renamed SWCLK
- net SWCLK: now also J27.5 (Pin_5)
- net swdio renamed SWDIO
- net SWDIO: now also J27.4 (Pin_4)
- no-connect marks 1 -> 3
Other:
- moved on the sheet: A1, C37, C38, C39, C40, C41, C42, C43, C44, C45, C46, C47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

Commit message: se agrego osciloscoio
Parts:
- removed J27: picoprobe debugger, Connector_PinHeader_2.54mm:PinHeader_1x07_P2.54mm_Vertical, symbol Connector:Conn_01x07_Pin
- added U10: W25Q16JVSS, kiC:Winbond_XSON-8-1EP_4x4mm_P0.8mm_EP2.3x3.0mm, symbol Memory_Flash:W25Q16JVSS
- SW7: value run -> boot; footprint Button_Switch_SMD:SW_SPST_B3U-1000P -> Button_Switch_SMD:SW_SPST_CK_RS282G05A3
Connections:
- net +3.3V: now also U10.8 (VCC)
- net GND: now also U10.4 (GND)
- net QSPI_CS: now also U10.1 (~{CS})
- net QSPI_SCLK: now also U10.6 (CLK)
- net QSPI_SD0: now also U10.5 (DI/IO_{0})
- net QSPI_SD1: now also U10.2 (DO/IO_{1})
- net QSPI_SD2: now also U10.3 (~{WP}/IO_{2})
- net QSPI_SD3: now also U10.7 (~{HOLD}/~{RESET}/IO_{3})
- no-connect marks 3 -> 1
