File: vga.kicad_sch (KiCad schematic)
At the start: 21 parts, among them J49 DE15_Pins_HighDensity

Commit message: se agrego osciloscoio
Connections:
- net GP_ renamed HSYNC
- net HSYNC: no longer R78.1
- net GP_0 renamed RED_0
- net GP_1 renamed RED_1
- net GP_10 renamed BLUE_4
- net GP_11 renamed BLUE_5
- net GP_12 renamed GREEN_0
- net GP_13 renamed GREEN_1
- net GP_14 renamed GREEN_2
- net GP_15 renamed GREEN_3
- net GP_16 renamed GREEN_4
- net GP_17 renamed GREEN_5
- net GP_2 renamed RED_2
- net GP_3 renamed RED_3
- net GP_4 renamed RED_4
- net GP_5 renamed RED_5
- net GP_6 renamed BLUE_0
- net GP_7 renamed BLUE_1
- net GP_8 renamed BLUE_2
- net GP_9 renamed BLUE_3
- new net VSYNC: R78.1
Changed lines of the file:
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@@
+	(wire
+		(pts
+			(xy 157.48 143.51) (xy 161.29 143.51)
+		)
+		(stroke
+			(width 0)
+			(type default)
+		)
+	)
 	(wire
 		(pts
@@
 		(pts
 			(xy 168.91 118.11) (xy 168.91 121.92)
-		)
-		(stroke
-			(width 0)
-			(type default)
-		)
-	)
-	(wire
-		(pts
-			(xy 157.48 143.51) (xy 161.29 143.51)
 		)
 		(stroke
@@
 		)
 	)
-	(hierarchical_label "GP_13"
+	(hierarchical_label "GREEN_2"
+		(shape input)
+		(at 157.48 143.51 180)
+		(effects
+			(font
+				(size 1.27 1.27)
+			)
+			(justify right)
+		)
+	)
+	(hierarchical_label "VSYNC"
+		(shape input)
+		(at 125.73 104.14 0)
+		(effects
+			(font
+				(size 1.27 1.27)
+			)
+			(justify left)
+		)
+	)
+	(hierarchical_label "RED_2"
+		(shape input)
+		(at 157.48 82.55 180)
+		(effects
+			(font
+				(size 1.27 1.27)
+			)
+			(justify right)
+		)
+	)
+	(hierarchical_label "GREEN_3"
+		(shape input)
+		(at 157.48 147.32 180)
+		(effects
+			(font
+				(size 1.27 1.27)
+			)
+			(justify right)
+		)
+	)
+	(hierarchical_label "GREEN_0"
+		(shape input)
+		(at 157.48 135.89 180)
+		(effects
+			(font
+				(size 1.27 1.27)
+			)
+			(justify right)
+		)
+	)
+	(hierarchical_label "BLUE_0"
+		(shape input)
+		(at 157.48 102.87 180)
+		(effects
+			(font
+				(size 1.27 1.27)
+			)
+			(justify right)
+		)
+	)
+	(hierarchical_label "RED_0"
+		(shape input)
+		(at 157.48 74.93 180)
+		(effects
+			(font
+				(size 1.27 1.27)
+			)
+			(justify right)
+		)
+	)
+	(hierarchical_label "RED_1"
+		(shape input)
+		(at 157.48 78.74 180)
+		(effects
+			(font
+				(size 1.27 1.27)
+			)
+			(justify right)
+		)
+	)
+	(hierarchical_label "BLUE_2"
+		(shape input)
+		(at 157.48 110.49 180)
+		(effects
+			(font
+				(size 1.27 1.27)
+			)
+			(justify right)
+		)
+	)
+	(hierarchical_label "GREEN_1"
 		(shape input)
 		(at 157.48 139.7 180)
@@
 		)
 	)
-	(hierarchical_label "GP_12"
-		(shape input)
-		(at 157.48 135.89 180)
-		(effects
-			(font
-				(size 1.27 1.27)
-			)
-			(justify right)
-		)
-	)
-	(hierarchical_label "GP_15"
-		(shape input)
-		(at 157.48 147.32 180)
-		(effects
-			(font
-				(size 1.27 1.27)
-			)
-			(justify right)
-		)
-	)
-	(hierarchical_label "GP_"
-		(shape input)
-		(at 125.73 104.14 0)
+	(hierarchical_label "RED_5"
+		(shape input)
+		(at 157.48 93.98 180)
+		(effects
+			(font
+				(size 1.27 1.27)
+			)
+			(justify right)
+		)
+	)
+	(hierarchical_label "GREEN_4"
+		(shape input)
+		(at 157.48 151.13 180)
+		(effects
+			(font
+				(size 1.27 1.27)
+			)
+			(justify right)
+		)
+	)
+	(hierarchical_label "BLUE_1"
+		(shape input)
+		(at 157.48 106.68 180)
+		(effects
+			(font
+				(size 1.27 1.27)
+			)
+			(justify right)
+		)
+	)
+	(hierarchical_label "BLUE_3"
+		(shape input)
+		(at 157.48 114.3 180)
+		(effects
+			(font
+				(size 1.27 1.27)
+			)
+			(justify right)
+		)
+	)
+	(hierarchical_label "RED_4"
+		(shape input)
+		(at 157.48 90.17 180)
+		(effects
+			(font
+				(size 1.27 1.27)
+			)
+			(justify right)
+		)
+	)
+	(hierarchical_label "HSYNC"
+		(shape input)
+		(at 125.73 109.22 0)
 		(effects
 			(font
@@
 		)
 	)
-	(hierarchical_label "GP_2"
-		(shape input)
-		(at 157.48 82.55 180)
-		(effects
-			(font
-				(size 1.27 1.27)
-			)
-			(justify right)
-		)
-	)
-	(hierarchical_label "GP_14"
-		(shape input)
-		(at 157.48 143.51 180)
-		(effects
-			(font
-				(size 1.27 1.27)
-			)
-			(justify right)
-		)
-	)
-	(hierarchical_label "GP_6"
-		(shape input)
-		(at 157.48 102.87 180)
-		(effects
-			(font
-				(size 1.27 1.27)
-			)
-			(justify right)
-		)
-	)
-	(hierarchical_label "GP_0"
-		(shape input)
-		(at 157.48 74.93 180)
-		(effects
-			(font
-				(size 1.27 1.27)
-			)
-			(justify right)
-		)
-	)
-	(hierarchical_label "GP_1"
-		(shape input)
-		(at 157.48 78.74 180)
-		(effects
-			(font
-				(size 1.27 1.27)
-			)
-			(justify right)
-		)
-	)
-	(hierarchical_label "GP_5"
-		(shape input)
-		(at 157.48 93.98 180)
-		(effects
-			(font
-				(size 1.27 1.27)
-			)
-			(justify right)
-		)
-	)
-	(hierarchical_label "GP_10"
+	(hierarchical_label "BLUE_4"
 		(shape input)
 		(at 157.48 118.11 180)
@@
 		)
 	)
-	(hierarchical_label "GP_17"
+	(hierarchical_label "GREEN_5"
 		(shape input)
 		(at 157.48 154.94 180)
@@
 		)
 	)
-	(hierarchical_label "GP_8"
-		(shape input)
-		(at 157.48 110.49 180)
-		(effects
-			(font
-				(size 1.27 1.27)
-			)
-			(justify right)
-		)
-	)
-	(hierarchical_label "GP_4"
-		(shape input)
-		(at 157.48 90.17 180)
-		(effects
-			(font
-				(size 1.27 1.27)
-			)
-			(justify right)
-		)
-	)
-	(hierarchical_label "GP_"
-		(shape input)
-		(at 125.73 109.22 0)
-		(effects
-			(font
-				(size 1.27 1.27)
-			)
-			(justify left)
-		)
-	)
-	(hierarchical_label "GP_9"
-		(shape input)
-		(at 157.48 114.3 180)
-		(effects
-			(font
-				(size 1.27 1.27)
-			)
-			(justify right)
-		)
-	)
-	(hierarchical_label "GP_11"
+	(hierarchical_label "BLUE_5"
 		(shape input)
 		(at 157.48 121.92 180)
@@
 		)
 	)
-	(hierarchical_label "GP_7"
-		(shape input)
-		(at 157.48 106.68 180)
-		(effects
-			(font
-				(size 1.27 1.27)
-			)
-			(justify right)
-		)
-	)
-	(hierarchical_label "GP_16"
-		(shape input)
-		(at 157.48 151.13 180)
-		(effects
-			(font
-				(size 1.27 1.27)
-			)
-			(justify right)
-		)
-	)
-	(hierarchical_label "GP_3"
+	(hierarchical_label "RED_3"
 		(shape input)
 		(at 157.48 86.36 180)
